File: Project_Final.kicad_pcb (KiCad board)
At the start: 2 copper layers, 72 x 98 mm, 56 parts, among them J1 Conn_01x02_Pin, J2 Conn_01x02_Pin, J3 Conn_01x02_Pin, J4 Conn_01x02_Pin, J5 Conn_01x02_Pin, Q1 2N3906, Q10 2N3906, Q11 2N3904, Q12 2N3906, Q13 2N3904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

Commit message: starting new layout
in progress
Parts:
- moved R1 71.5 mm to (110.2, 20.7)
- moved R2 71.5 mm to (125.9, 20.5)
- moved Q15 46.6 mm to (24.7, 92.9), turned to 90 degrees
- moved Q18 45.7 mm to (24.1, 97.7), turned to -90 degrees
- moved Q19 37.7 mm to (33.4, 92.8), turned to 90 degrees
- moved Q20 36.9 mm to (33.1, 97.7), turned to -90 degrees
- moved Q22 34.2 mm to (41.9, 100.3), turned to 90 degrees
- moved Q21 31.2 mm to (41.5, 90.5), turned to -90 degrees
- moved R13 28.9 mm to (70.7, 88.8)
- moved R14 28.7 mm to (75.2, 88.8)
- moved R6 28.6 mm to (79.7, 88.8)
- moved J3 27.3 mm to (108.0, 57.5)
- moved J4 27.3 mm to (108.0, 52.0)
- moved R5 17.1 mm to (82.0, 19.8)
- moved Q7 16.9 mm to (76.9, 31.0)
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Connections:
- C3 pad 2: Vee -> VEE
Routing:
- net Vee: track 152.7 -> 0.00 mm
- net VCC: track 132.8 -> 0.00 mm
- net V_Out_Output: track 86.3 -> 0.00 mm
- net V_In_Output: track 80.1 -> 0.00 mm
- net V_Out_Op-Amp: track 66.0 -> 0.00 mm
- net V-: track 56.2 -> 0.00 mm
- net Net-(J2-Pin_1): track 39.8 -> 0.00 mm
- net Net-(Q5-C): track 34.8 -> 0.00 mm
- net VEE: track 28.7 -> 0.00 mm
- net V+: track 27.2 -> 0.00 mm
- net Net-(Q1-B): track 22.5 -> 0.00 mm
- net Net-(Q10-B): track 21.2 -> 0.00 mm
- net Net-(Q14-C): track 20.6 -> 0.00 mm
- net Net-(C2-Pad2): track 20.5 -> 0.00 mm
- net Net-(Q2-E): track 19.8 -> 0.00 mm
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Other:
- board size 72 x 98 mm -> 72 x 111.5 mm

Commit message: edits. near final layout
Parts:
- removed the R1 at (88.0, 36.8)
- removed the TP1 at (102.0, 76.5)
- moved R1 73.8 mm to (108.6, 94.6), turned to -90 degrees
- moved Q15 63.7 mm to (77.6, 57.4), turned to 0 degrees
- moved Q18 63.5 mm to (72.8, 56.9), turned to 180 degrees
- moved R12 63.1 mm to (84.0, 65.5), turned to 90 degrees
- moved R16 61.6 mm to (84.0, 68.7), turned to -90 degrees
- moved R2 60.6 mm to (108.6, 78.5), turned to -90 degrees
- moved CPaddle1 59.9 mm to (88.5, 86.0), turned to 180 degrees
- moved TP1 54.9 mm to (100.5, 69.5)
- moved JPaddle1 53.8 mm to (94.0, 69.5)
- moved Q19 51.8 mm to (77.7, 66.1), turned to 0 degrees
- moved Q20 50.9 mm to (72.8, 65.9), turned to 180 degrees
- moved R17 47.2 mm to (65.5, 81.2), turned to 90 degrees
- moved Q21 41.8 mm to (80.0, 74.2), turned to 180 degrees
- moved R15 41.6 mm to (65.5, 54.0), turned to -90 degrees
- moved Q22 38.3 mm to (70.2, 74.6), turned to 0 degrees
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Routing:
- added copper zone on F.Cu, net VEE
- removed copper zone on F.Cu, net Net-(J1-Pin_1)
Other:
- board size 72 x 111.5 mm -> 73.5 x 111.5 mm

Commit message: finished layout
Parts:
- TP1: footprint Connector_Pin:Pin_D1.0mm_L10.0mm -> Library:Single_Relief
- moved J4 41.0 mm to (94.8, 87.3), turned to 0 degrees
- moved R13 40.1 mm to (67.8, 48.8)
- moved R14 40.1 mm to (72.3, 48.8)
- moved R6 39.9 mm to (77.1, 48.9)
- moved TP1 33.1 mm to (131.8, 59.0), turned to 90 degrees
- moved CPaddle1 32.6 mm to (104.9, 57.8), turned to 90 degrees
- moved J3 30.4 mm to (94.7, 81.5)
- moved JTestPoint1 27.0 mm to (112.1, 86.5)
- moved RLoad1 27.0 mm to (117.1, 88.5)
- moved C2 26.9 mm to (104.2, 87.7)
- moved JPaddle1 21.5 mm to (112.2, 57.9), turned to -90 degrees
- moved J2 20.2 mm to (94.7, 75.9)
- moved R1 15.7 mm to (105.9, 79.1), turned to 0 degrees
- moved Q13 13.8 mm to (72.7, 93.6)
- moved Q10 13.5 mm to (75.3, 106.4)
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Routing:
- added copper zone on B.Cu, net VEE
Other:
- board size 73.5 x 111.5 mm -> 70.4 x 107.1 mm

Commit message: finished
Parts:
- added G***: LOGO, Library:cat-image, F.Cu at (117.5, 33.5)
- moved R10 15.0 mm to (87.2, 105.5), turned to 0 degrees
- moved J4 9.83 mm to (96.0, 77.5)
- moved J1 9.83 mm to (95.9, 60.6)
- moved J2 9.83 mm to (95.9, 66.1)
- moved J3 9.83 mm to (95.9, 71.7)
- moved Q8 8.51 mm to (96.3, 30.6), turned to 180 degrees
- moved CByPass1 8.48 mm to (94.8, 90.2)
- moved J5 8.48 mm to (95.0, 96.0)
- moved Q1 5.09 mm to (71.5, 39.5)
- moved Q3 5.09 mm to (77.0, 39.5)
- moved Q6 5.09 mm to (82.9, 39.7)
- moved Q9 5.09 mm to (88.3, 39.7)
- moved R3 4.88 mm to (85.0, 44.0)
- moved R4 4.88 mm to (89.5, 55.7)
- moved R13 4.86 mm to (68.6, 44.0)
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Routing:
- net V-: track 0.00 -> 71.0 mm
- net V_Out_Output: track 0.00 -> 55.4 mm
- net V+: track 0.00 -> 53.9 mm
- net Net-(J2-Pin_1): track 0.00 -> 52.9 mm
- net V_Out_Op-Amp: track 0.00 -> 50.6 mm
- net Net-(Q15-E): track 0.00 -> 50.5 mm, vias 0 -> 1
- net V_In_Output: track 0.00 -> 45.7 mm
- net Net-(Q5-C): track 0.00 -> 32.5 mm
- net Net-(J3-Pin_1): track 0.00 -> 30.0 mm
- net Net-(JBattery1-Pin_1): track 0.00 -> 24.9 mm
- net Net-(Q1-B): track 0.00 -> 22.9 mm
- net Net-(Q10-B): track 0.00 -> 21.7 mm
- net Net-(J1-Pin_1): track 0.00 -> 20.4 mm
- net Net-(Q19-C): track 0.00 -> 18.7 mm
- net Net-(Q15-B): track 0.00 -> 17.4 mm
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- added copper zone on F.Cu, net VCC
Other:
- board text added: "Speaker"

Commit message: fixed Errors
Routing:
- net Net-(Q20-C): track 0.00 -> 18.3 mm
Changed lines of the file:
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@@
 		(tags "to-92 sc-43 sc-43a sot54 PA33 transistor")
 		(property "Reference" "Q7"
-			(at 1.27 -1.5 90)
+			(at 1.27 -1.5 180)
 			(layer "F.SilkS")
 			(effects
@@
 		(tags "to-92 sc-43 sc-43a sot54 PA33 transistor")
 		(property "Reference" "Q21"
-			(at 1.27 -3.56 0)
+			(at 1.23566 2.83711 0)
 			(layer "F.SilkS")
 			(effects
@@
 		(tags "to-92 sc-43 sc-43a sot54 PA33 transistor")
 		(property "Reference" "Q1"
-			(at 1.27 -2 90)
+			(at 1.234133 -1.522807 180)
 			(layer "F.SilkS")
 			(effects
@@
 		(tags "to-92 sc-43 sc-43a sot54 PA33 transistor")
 		(property "Reference" "Q9"
-			(at 1.27 -1.36 90)
+			(at 1.27 -1.36 180)
 			(layer "F.SilkS")
 			(effects
@@
 		(tags "to-92 sc-43 sc-43a sot54 PA33 transistor")
 		(property "Reference" "Q20"
-			(at 1.27 -3.56 0)
+			(at 1.27 2.702568 0)
 			(layer "F.SilkS")
 			(effects
@@
 		(tags "to-92 sc-43 sc-43a sot54 PA33 transistor")
 		(property "Reference" "Q2"
-			(at 1.27 -1.86 90)
+			(at 1.27 -1.86 180)
 			(layer "F.SilkS")
 			(effects
@@
 		(tags "to-92 sc-43 sc-43a sot54 PA33 transistor")
 		(property "Reference" "Q6"
-			(at 1.27 -2 90)
+			(at 1.27 -1.541037 180)
 			(layer "F.SilkS")
 			(effects
@@
 		(tags "to-92 sc-43 sc-43a sot54 PA33 transistor")
 		(property "Reference" "Q3"
-			(at 1.27 -2 90)
+			(at 1.27 -1.63725 180)
 			(layer "F.SilkS")
 			(effects
@@
 		(tags "to-92 sc-43 sc-43a sot54 PA33 transistor")
 		(property "Reference" "Q18"
-			(at 1.27 -3.56 0)
+			(at 1.378634 2.690385 0)
 			(layer "F.SilkS")
 			(effects
@@
 		(net 28)
 	)
+	(segment
+		(start 74.05 74.26)
+		(end 74.05 81.21)
+		(width 0.2)
+		(layer "F.Cu")
+		(net 29)
+	)
+	(segment
+		(start 72.78 72.99)
+		(end 74.05 74.26)
+		(width 0.2)
+		(layer "F.Cu")
+		(net 29)
+	)
+	(segment
+		(start 74.05 81.21)
+		(end 74.05 81.872)
+		(width 0.2)
+		(layer "F.Cu")
+		(net 29)
+	)
+	(segment
+		(start 74.05 81.872)
+		(end 68.1 87.822)
+		(width 0.2)
+		(layer "F.Cu")
+		(net 29)
+	)
+	(segment
+		(start 72.78 72.49)
+		(end 72.78 72.99)
+		(width 0.2)
+		(layer "F.Cu")
+		(net 29)
+	)
 	(zone

Commit message: updated
Parts:
- C1, C3, CByPass1, CPaddle1: footprint ECA_1HHG330:CAPPRD200W50D500H1100 -> Capacitor_THT:C_Radial_D5.0mm_H11.0mm_P2.00mm
- R1, R2: footprint 35ZLH100MEFC6_3X11:PTV09A-4015F-B104_BRN -> footprints:PTV09A-4015F-B104_BRN
- moved C1 1.00 mm to (96.0, 37.5)
- moved C3 1.00 mm to (96.0, 44.0)
- moved CPaddle1 1.00 mm to (105.5, 59.0)
- moved CByPass1 0.85 mm to (94.0, 90.2)
Routing:
- net V_Out_Output: track 55.4 -> 58.6 mm
Other:
- board text added: "Q12"
