File: Op-Amp.kicad_sch (KiCad schematic)
At the start: 26 parts, among them Q1 2N3906, Q15 2N3906, Q18 2N3904, Q19 2N3906, Q2 2N3906, Q20 2N3904, Q21 2N3904, Q22 2N3906, Q3 2N3906, Q4 2N3904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

Commit message: update with john's copy
Connections:
- net Vee: no longer Q22.1 (E), Q4.1 (E), Q5.1 (E), R11.1, R15.2, R17.2, R5.1
- net Vcc renamed VCC
- new net VEE: Q22.1 (E), Q4.1 (E), Q5.1 (E), R11.1, R15.2, R17.2, R5.1

Commit message: starting new layout
in progress
Connections:
- net Vee is gone; now on net VEE: C3.2
Changed lines of the file:
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@@
 (kicad_sch
-	(version 20231120)
+	(version 20250114)
 	(generator "eeschema")
-	(generator_version "8.0")
+	(generator_version "9.0")
 	(paper "A4")
 	(junction
@@
 		)
 	)
-	(global_label "Vee"
-		(shape input)
-		(at 109.22 59.69 270)
-		(fields_autoplaced yes)
-		(effects
-			(font
-				(size 1.27 1.27)
-			)
-			(justify right)
-		)
-		(property "Intersheetrefs" "${INTERSHEET_REFS}"
-			(at 109.22 65.941 90)
-			(effects
-				(font
-					(size 1.27 1.27)
-				)
-				(justify right)
-				(hide yes)
-			)
-		)
-	)
 	(global_label "V_Out_Op-Amp"
 		(shape input)
@@
 					(unit 1)
 				)
+			)
+		)
+	)
+	(symbol
+		(lib_id "power:VEE")
+		(at 109.22 59.69 180)
+		(unit 1)
+		(exclude_from_sim no)
+		(in_bom yes)
+		(on_board yes)
+		(dnp no)
+		(fields_autoplaced yes)
+		(property "Reference" "#PWR015"
+			(at 109.22 55.88 0)
+			(effects
+				(font
+					(size 1.27 1.27)
+				)
+				(hide yes)
+			)
+		)
+		(property "Value" "VEE"
+			(at 109.22 64.77 0)
+			(effects
+				(font
+					(size 1.27 1.27)
+				)
+			)
+		)
+		(property "Footprint" ""
+			(at 109.22 59.69 0)
+			(effects
+				(font
+					(size 1.27 1.27)
+				)
+				(hide yes)
+			)
+		)
+		(property "Datasheet" ""
+			(at 109.22 59.69 0)
+			(effects
+				(font
+					(size 1.27 1.27)
+				)
+				(hide yes)
+			)
+		)
+		(property "Description" "Power symbol creates a global label with name \"VEE\""
+			(at 109.22 59.69 0)
+			(effects
+				(font
+					(size 1.27 1.27)
+				)
+				(hide yes)
+			)
+		)
+		(pin "1"
+		)
+		(instances
+			(project "Project_Final"
+				(path "/ae7489fb-4acd-4c47-9498-30070a4fb91b/d35e8965-c723-4eb0-9f76-96e1d82904a7"
+					(reference "#PWR015")
+					(unit 1)
+				)

Commit message: updated
Parts:
- C1, C3: footprint ECA_1HHG330:CAPPRD200W50D500H1100 -> Capacitor_THT:C_Radial_D5.0mm_H11.0mm_P2.00mm
Changed lines of the file:
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@@
 			)
 		)
-		(property "Footprint" "ECA_1HHG330:CAPPRD200W50D500H1100"
+		(property "Footprint" "Capacitor_THT:C_Radial_D5.0mm_H11.0mm_P2.00mm"
 			(at 110.1852 59.69 0)
 			(effects
@@
 			)
 		)
-		(property "Footprint" "ECA_1HHG330:CAPPRD200W50D500H1100"
+		(property "Footprint" "Capacitor_THT:C_Radial_D5.0mm_H11.0mm_P2.00mm"
 			(at 117.8052 53.34 0)
 			(effects

Commit message: updated values
Parts:
- C1: value C -> 0
- C3: value C -> 100n
- R11: value R -> 5.5k
- R12, R15, R16, R17: value R -> 4.7k
- R13, R5, R6: value R -> 390
- R14: value R -> 180
Changed lines of the file:
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@@
 			)
 		)
-		(property "Value" "R"
+		(property "Value" "5.5k"
 			(at 33.02 24.1299 0)
 			(effects
@@
 			)
 		)
-		(property "Value" "R"
+		(property "Value" "180"
 			(at 85.09 87.6299 0)
 			(effects
@@
 			)
 		)
-		(property "Value" "R"
+		(property "Value" "4.7k"
 			(at 214.63 135.8899 0)
 			(effects
@@
 			)
 		)
-		(property "Value" "R"
+		(property "Value" "4.7k"
 			(at 187.96 81.2799 0)
 			(effects
@@
 			)
 		)
-		(property "Value" "R"
+		(property "Value" "390"
 			(at 127 87.6299 0)
 			(effects
@@
 			)
 		)
-		(property "Value" "R"
+		(property "Value" "4.7k"
 			(at 187.96 129.5399 0)
 			(effects
@@
 			)
 		)
-		(property "Value" "R"
+		(property "Value" "4.7k"
 			(at 204.47 77.4699 0)
 			(effects
@@
 			)
 		)
-		(property "Value" "C"
+		(property "Value" "100n"
 			(at 112.522 59.182 0)
 			(effects
@@
 			)
 		)
-		(property "Value" "C"
+		(property "Value" "0"
 			(at 120.65 50.7999 0)
 			(effects
@@
 			)
 		)
-		(property "Value" "R"
+		(property "Value" "390"
 			(at 127 24.1299 0)
 			(effects
@@
 			)
 		)
-		(property "Value" "R"
+		(property "Value" "390"
 			(at 34.29 87.6299 0)
 			(effects
