File: Output AB Buffer Stage.kicad_sch (KiCad schematic)
At the start: 10 parts, among them Q10 2N3906, Q11 2N3904, Q12 2N3906, Q13 2N3904, Q14 2N3904, Q16 2N3906

Commit message: update with john's copy
Connections:
- net Vcc renamed VCC
- net Vee renamed VEE
Changed lines of the file:
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@@
+	)
+	(junction
+		(at 90.17 50.8)
+		(diameter 0)
+		(color 0 0 0 0)
 	)
 	(junction
@@
 	)
 	(junction
+		(at 93.98 133.35)
+		(diameter 0)
+		(color 0 0 0 0)
+	)
+	(junction
 		(at 71.12 80.01)
 		(diameter 0)
@@
 	(wire
 		(pts
+			(xy 93.98 133.35) (xy 97.79 133.35)
+		)
+		(stroke
+			(width 0)
+			(type default)
+		)
+	)
+	(wire
+		(pts
 			(xy 87.63 58.42) (xy 87.63 60.96)
 		)
@@
 	(wire
 		(pts
-			(xy 87.63 50.8) (xy 111.76 50.8)
+			(xy 87.63 50.8) (xy 90.17 50.8)
 		)
 		(stroke
@@
 	(wire
 		(pts
+			(xy 90.17 50.8) (xy 111.76 50.8)
+		)
+		(stroke
+			(width 0)
+			(type default)
+		)
+	)
+	(wire
+		(pts
 			(xy 96.52 88.9) (xy 96.52 92.71)
 		)
@@
 	(wire
 		(pts
-			(xy 71.12 133.35) (xy 97.79 133.35)
+			(xy 71.12 133.35) (xy 93.98 133.35)
 		)
 		(stroke
@@
 		)
 	)
-	(global_label "Vee"
-		(shape input)
-		(at 97.79 133.35 270)
-		(fields_autoplaced yes)
-		(effects
-			(font
-				(size 1.27 1.27)
-			)
-			(justify right)
-		)
-		(property "Intersheetrefs" "${INTERSHEET_REFS}"
-			(at 97.79 139.601 90)
-			(effects
-				(font
-					(size 1.27 1.27)
-				)
-				(justify right)
-				(hide yes)
-			)
-		)
-	)
-	(global_label "Vcc"
-		(shape input)
-		(at 87.63 50.8 90)
-		(fields_autoplaced yes)
-		(effects
-			(font
-				(size 1.27 1.27)
-			)
-			(justify left)
-		)
-		(property "Intersheetrefs" "${INTERSHEET_REFS}"
-			(at 87.63 44.549 90)
-			(effects
-				(font
-					(size 1.27 1.27)
-				)
-				(justify left)
-				(hide yes)
-			)
-		)
-	)
 	(global_label "V_In_Output"
 		(shape input)
@@
 				(justify right)
 				(hide yes)
+			)
+		)
+	)
+	(symbol
+		(lib_id "power:VEE")
+		(at 93.98 133.35 180)
+		(unit 1)
+		(exclude_from_sim no)
+		(in_bom yes)
+		(on_board yes)
+		(dnp no)
+		(fields_autoplaced yes)
+		(property "Reference" "#PWR014"
+			(at 93.98 129.54 0)
+			(effects
+				(font
+					(size 1.27 1.27)
+				)
+				(hide yes)
+			)
+		)
+		(property "Value" "VEE"
+			(at 93.98 138.43 0)
+			(effects
+				(font
+					(size 1.27 1.27)
+				)
+			)
+		)
+		(property "Footprint" ""
+			(at 93.98 133.35 0)
+			(effects
+				(font
+					(size 1.27 1.27)
+				)
+				(hide yes)
+			)
+		)
+		(property "Datasheet" ""
+			(at 93.98 133.35 0)
+			(effects
+				(font
+					(size 1.27 1.27)
+				)
+				(hide yes)
+			)
+		)
+		(property "Description" "Power symbol creates a global label with name \"VEE\""
+			(at 93.98 133.35 0)
+			(effects
+				(font
+					(size 1.27 1.27)
+				)
+				(hide yes)
+			)
+		)
+		(pin "1"
+		)
+		(instances
+			(project "ECE 3660 Design Project"
+				(path "/ae7489fb-4acd-4c47-9498-30070a4fb91b/85fa7e5a-922a-4eb2-9c5d-36a4e560037a"
+					(reference "#PWR014")
+					(unit 1)
+				)
 			)
 		)
@@
 					(unit 1)
 				)
+			)
+		)
+	)
+	(symbol
+		(lib_id "power:VCC")
+		(at 90.17 50.8 0)
+		(unit 1)
+		(exclude_from_sim no)
+		(in_bom yes)
+		(on_board yes)
+		(dnp no)
+		(fields_autoplaced yes)
+		(property "Reference" "#PWR013"
+			(at 90.17 54.61 0)
+			(effects
+				(font
+					(size 1.27 1.27)
+				)
+				(hide yes)
+			)
+		)
+		(property "Value" "VCC"
+			(at 90.17 45.72 0)
+			(effects
+				(font
+					(size 1.27 1.27)
+				)
+			)
+		)
+		(property "Footprint" ""
+			(at 90.17 50.8 0)
+			(effects
+				(font
+					(size 1.27 1.27)
+				)
+				(hide yes)
+			)
+		)
+		(property "Datasheet" ""
+			(at 90.17 50.8 0)
+			(effects
+				(font
+					(size 1.27 1.27)
+				)
+				(hide yes)
+			)
+		)
+		(property "Description" "Power symbol creates a global label with name \"VCC\""
+			(at 90.17 50.8 0)
+			(effects
+				(font
+					(size 1.27 1.27)
+				)
+				(hide yes)
+			)
+		)
+		(pin "1"
+		)
+		(instances
+			(project "ECE 3660 Design Project"
+				(path "/ae7489fb-4acd-4c47-9498-30070a4fb91b/85fa7e5a-922a-4eb2-9c5d-36a4e560037a"
+					(reference "#PWR013")
+					(unit 1)
+				)

Commit message: updated values
Parts:
- R10, R9: value R -> 22k
- R7, R8: value R -> 4.7k
Changed lines of the file:
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@@
 			)
 		)
-		(property "Value" "R"
+		(property "Value" "4.7k"
 			(at 100.33 114.2999 0)
 			(effects
@@
 			)
 		)
-		(property "Value" "R"
+		(property "Value" "4.7k"
 			(at 90.17 55.8799 0)
 			(effects
@@
 			)
 		)
-		(property "Value" "R"
+		(property "Value" "22k"
 			(at 73.66 107.9499 0)
 			(effects
@@
 			)
 		)
-		(property "Value" "R"
+		(property "Value" "22k"
 			(at 73.66 59.6899 0)
 			(effects
