File: Project_Final.kicad_sch (KiCad schematic)
At the start: 18 parts, among them J1 Conn_01x02_Pin, J2 Conn_01x02_Pin, J3 Conn_01x02_Pin, J4 Conn_01x02_Pin, J5 Conn_01x02_Pin, Q17 BSP89

Commit message: update with john's copy
Connections:
- net V-: now also R1.3; no longer R1.2
- net VEE: now also JPaddle1.1 (Pin_1)
- net V_Out_Op-Amp: now also R1.2
- net at CPaddle1.1, J1.1 (Pin_1), TP1.1: now also JPaddle1.2 (Pin_2)
- net at J2.1 (Pin_1), R3.2, R4.1: now also R2.3; no longer R2.2
- net at J3.1 (Pin_1), R2.1: now also R2.2
Other:
- moved on the sheet: JPaddle1, TP1

Commit message: finished layout
Parts:
- TP1: footprint Connector_Pin:Pin_D1.0mm_L10.0mm -> Library:Single_Relief
Changed lines of the file:
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@@
 		(dnp no)
 		(property "Reference" "TP1"
-			(at 36.322 43.942 90)
+			(at 34.29 43.942 90)
 			(effects
 				(font
@@
 		)
 		(property "Value" "TestPoint"
-			(at 37.592 45.974 90)
+			(at 32.512 46.228 90)
 			(effects
 				(font
@@
 			)
 		)
-		(property "Footprint" "Connector_Pin:Pin_D1.0mm_L10.0mm"
+		(property "Footprint" "Library:Single_Relief"
 			(at 33.02 53.34 0)
 			(effects

Commit message: updated
Parts:
- CByPass1, CPaddle1: footprint ECA_1HHG330:CAPPRD200W50D500H1100 -> Capacitor_THT:C_Radial_D5.0mm_H11.0mm_P2.00mm
Changed lines of the file:
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@@
 			)
 		)
-		(property "Footprint" "ECA_1HHG330:CAPPRD200W50D500H1100"
+		(property "Footprint" "Capacitor_THT:C_Radial_D5.0mm_H11.0mm_P2.00mm"
 			(at 26.3652 29.21 0)
 			(effects
@@
 			)
 		)
-		(property "Footprint" "ECA_1HHG330:CAPPRD200W50D500H1100"
+		(property "Footprint" "Capacitor_THT:C_Radial_D5.0mm_H11.0mm_P2.00mm"
 			(at 101.2952 134.62 0)
 			(effects

Commit message: updated values
Parts:
- R3, R4: value R -> 100k
Changed lines of the file:
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@@
 			)
 		)
-		(property "Value" "R"
+		(property "Value" "100k"
 			(at 45.72 54.6099 0)
 			(effects
@@
 			)
 		)
-		(property "Value" "R"
+		(property "Value" "100k"
 			(at 45.72 44.4499 0)
 			(effects
